Commit message: Update parameters and configs

File: legged_perceptive_description/urdf/gazebo_d400.xacro (robot description, xacro)
@@ -94,5 +94,5 @@
                     <clip>
                         <near>0.1</near>
-                        <far>100</far>
+                        <far>5</far>
                     </clip>
                     <noise>

File: legged_perceptive_description/urdf/robot.xacro (robot description, xacro)
@@ -5,9 +5,9 @@
     <xacro:include filename="$(find legged_perceptive_description)/urdf/sensor_d435.xacro"/>
     <xacro:include filename="$(find legged_perceptive_description)/urdf/sensor_t265.xacro"/>
+    <xacro:sensor_d435 name="front_camera" topics_ns="front_camera" parent="base">
+        <origin xyz="0.305 0 -0.04" rpy="0 0.25 0"/>
+    </xacro:sensor_d435>
     <xacro:sensor_t265 name="tracking_camera" topics_ns="tracking_camera" parent="base">
-        <origin xyz="-0.068 0 0.142" rpy="1.5707 -1.8324 0"/>
+        <origin xyz="0.33 0.01 0" rpy="0 0.25 0"/>
     </xacro:sensor_t265>
-    <xacro:sensor_d435 name="front_camera" topics_ns="front_camera" parent="base">
-        <origin xyz="0.35 0 0.1" rpy="0 0.52 0"/>
-    </xacro:sensor_d435>
 </robot>

Commit message: Update camera pose

File: legged_perceptive_description/urdf/gazebo_d400.xacro (robot description, xacro)
@@ -103,5 +103,5 @@
                 </camera>
                 <always_on>1</always_on>
-                <update_rate>5</update_rate>
+                <update_rate>10</update_rate>
                 <visualize>0</visualize>
             </sensor>

File: legged_perceptive_description/urdf/robot.xacro (robot description, xacro)
@@ -6,5 +6,5 @@
     <xacro:include filename="$(find legged_perceptive_description)/urdf/sensor_t265.xacro"/>
     <xacro:sensor_d435 name="front_camera" topics_ns="front_camera" parent="base">
-        <origin xyz="0.349 0.021 -0.035" rpy="0 0.872 0"/>
+        <origin xyz="0.349 0.021 -0.035" rpy="1.57 0.64 0"/>
     </xacro:sensor_d435>
     <xacro:sensor_t265 name="tracking_camera" topics_ns="tracking_camera" parent="base">
