Commit message: Update parameters and configs

File: legged_perceptive_description/urdf/robot.xacro (robot description, xacro)
@@ -6,8 +6,8 @@
     <xacro:include filename="$(find legged_perceptive_description)/urdf/sensor_t265.xacro"/>
     <xacro:sensor_d435 name="front_camera" topics_ns="front_camera" parent="base">
-        <origin xyz="0.349 0.021 -0.035" rpy="0 0.872 0"/>
+        <origin xyz="0.305 0 -0.04" rpy="0 0.25 0"/>
     </xacro:sensor_d435>
     <xacro:sensor_t265 name="tracking_camera" topics_ns="tracking_camera" parent="base">
-        <origin xyz="0.387 0.01 0.002" rpy="0 0 0"/>
+        <origin xyz="0.33 0.01 0" rpy="0 0.25 0"/>
     </xacro:sensor_t265>
 </robot>

Commit message: Add unitree_hw.launch

File: legged_perceptive_description/urdf/robot.xacro (robot description, xacro)
@@ -6,8 +6,8 @@
     <xacro:include filename="$(find legged_perceptive_description)/urdf/sensor_t265.xacro"/>
     <xacro:sensor_d435 name="front_camera" topics_ns="front_camera" parent="base">
-        <origin xyz="0.305 0 -0.04" rpy="0 0.25 0"/>
+        <origin xyz="0.305 0.01 -0.07" rpy="-0.025 0.25 0"/>
     </xacro:sensor_d435>
     <xacro:sensor_t265 name="tracking_camera" topics_ns="tracking_camera" parent="base">
-        <origin xyz="0.33 0.01 0" rpy="0 0.25 0"/>
+        <origin xyz="0.33 0.01 0" rpy="0 0.22 0"/>
     </xacro:sensor_t265>
 </robot>

Commit message: First experience config that work!

File: legged_perceptive_description/urdf/robot.xacro (robot description, xacro)
@@ -6,8 +6,8 @@
     <xacro:include filename="$(find legged_perceptive_description)/urdf/sensor_t265.xacro"/>
     <xacro:sensor_d435 name="front_camera" topics_ns="front_camera" parent="base">
-        <origin xyz="0.305 0.01 -0.07" rpy="-0.025 0.25 0"/>
+        <origin xyz="0.29 0.01 -0.05" rpy="-0.02 0.22 0"/>
     </xacro:sensor_d435>
     <xacro:sensor_t265 name="tracking_camera" topics_ns="tracking_camera" parent="base">
-        <origin xyz="0.33 0.01 0" rpy="0 0.22 0"/>
+        <origin xyz="0.32 0.01 0" rpy="0 0.25 0"/>
     </xacro:sensor_t265>
 </robot>

Commit message: First experience config that work!

File: legged_perceptive_description/urdf/robot.xacro (robot description, xacro)
@@ -6,8 +6,8 @@
     <xacro:include filename="$(find legged_perceptive_description)/urdf/sensor_t265.xacro"/>
     <xacro:sensor_d435 name="front_camera" topics_ns="front_camera" parent="base">
-        <origin xyz="0.349 0.021 -0.035" rpy="0 0.872 0"/>
+        <origin xyz="0.29 0.01 -0.05" rpy="-0.02 0.22 0"/>
     </xacro:sensor_d435>
     <xacro:sensor_t265 name="tracking_camera" topics_ns="tracking_camera" parent="base">
-        <origin xyz="0.387 0.01 0.002" rpy="0 0 0"/>
+        <origin xyz="0.32 0.01 0" rpy="0 0.25 0"/>
     </xacro:sensor_t265>
 </robot>

Commit message: Update camera pose

File: legged_perceptive_description/urdf/robot.xacro (robot description, xacro)
@@ -6,8 +6,8 @@
     <xacro:include filename="$(find legged_perceptive_description)/urdf/sensor_t265.xacro"/>
     <xacro:sensor_d435 name="front_camera" topics_ns="front_camera" parent="base">
-        <origin xyz="0.29 0.01 -0.05" rpy="-0.02 0.22 0"/>
+        <origin xyz="0.349 0.021 -0.035" rpy="0 0.872 0"/>
     </xacro:sensor_d435>
     <xacro:sensor_t265 name="tracking_camera" topics_ns="tracking_camera" parent="base">
-        <origin xyz="0.32 0.01 0" rpy="0 0.25 0"/>
+        <origin xyz="0.387 0.01 0.002" rpy="0 0 0"/>
     </xacro:sensor_t265>
 </robot>

Commit message: Update camera pose

File: legged_perceptive_description/urdf/robot.xacro (robot description, xacro)
@@ -6,8 +6,8 @@
     <xacro:include filename="$(find legged_perceptive_description)/urdf/sensor_t265.xacro"/>
     <xacro:sensor_d435 name="front_camera" topics_ns="front_camera" parent="base">
-        <origin xyz="0.29 0.01 -0.05" rpy="-0.02 0.22 0"/>
+        <origin xyz="0.349 0.021 -0.035" rpy="1.57 0.64 0"/>
     </xacro:sensor_d435>
     <xacro:sensor_t265 name="tracking_camera" topics_ns="tracking_camera" parent="base">
-        <origin xyz="0.32 0.01 0" rpy="0 0.25 0"/>
+        <origin xyz="0.387 0.01 0.002" rpy="0 0 0"/>
     </xacro:sensor_t265>
 </robot>

Commit message: Update camera pose

File: legged_perceptive_description/urdf/robot.xacro (robot description, xacro)
@@ -6,8 +6,8 @@
     <xacro:include filename="$(find legged_perceptive_description)/urdf/sensor_t265.xacro"/>
     <xacro:sensor_d435 name="front_camera" topics_ns="front_camera" parent="base">
-        <origin xyz="0.349 0.021 -0.035" rpy="1.57 0.64 0"/>
+        <origin xyz="0.36 -0.0 0.03" rpy="3.1415 0.4 0"/>
     </xacro:sensor_d435>
     <xacro:sensor_t265 name="tracking_camera" topics_ns="tracking_camera" parent="base">
-        <origin xyz="0.387 0.01 0.002" rpy="0 0 0"/>
+        <origin xyz="0.15 0 0.1" rpy="0 -1.04 0"/>
     </xacro:sensor_t265>
 </robot>

Commit message: Update parameters

File: legged_perceptive_description/urdf/robot.xacro (robot description, xacro)
@@ -6,8 +6,8 @@
     <xacro:include filename="$(find legged_perceptive_description)/urdf/sensor_t265.xacro"/>
     <xacro:sensor_d435 name="front_camera" topics_ns="front_camera" parent="base">
-        <origin xyz="0.36 -0.0 0.03" rpy="3.1415 0.4 0"/>
+        <origin xyz="0.36 -0.0 0.02" rpy="3.16 0.4 0"/>
     </xacro:sensor_d435>
     <xacro:sensor_t265 name="tracking_camera" topics_ns="tracking_camera" parent="base">
-        <origin xyz="0.15 0 0.1" rpy="0 -1.04 0"/>
+        <origin xyz="0.145 0 0.1" rpy="0 -1.04 0"/>
     </xacro:sensor_t265>
 </robot>

Commit message: Update camera pose

File: legged_perceptive_description/urdf/robot.xacro (robot description, xacro)
@@ -6,5 +6,5 @@
     <xacro:include filename="$(find legged_perceptive_description)/urdf/sensor_t265.xacro"/>
     <xacro:sensor_d435 name="front_camera" topics_ns="front_camera" parent="base">
-        <origin xyz="0.36 -0.0 0.02" rpy="3.16 0.4 0"/>
+        <origin xyz="0.36 -0.0 0.01" rpy="3.141 0.38 0"/>
     </xacro:sensor_d435>
     <xacro:sensor_t265 name="tracking_camera" topics_ns="tracking_camera" parent="base">

Commit message: Add mid360 launch

File: legged_perceptive_description/urdf/robot.xacro (robot description, xacro)
@@ -5,9 +5,28 @@
     <xacro:include filename="$(find legged_perceptive_description)/urdf/sensor_d435.xacro"/>
     <xacro:include filename="$(find legged_perceptive_description)/urdf/sensor_t265.xacro"/>
-    <xacro:sensor_d435 name="front_camera" topics_ns="front_camera" parent="base">
-        <origin xyz="0.36 -0.0 0.01" rpy="3.141 0.38 0"/>
-    </xacro:sensor_d435>
+    <!--    <xacro:sensor_d435 name="front_camera" topics_ns="front_camera" parent="base">-->
+    <!--        <origin xyz="0.36 -0.0 0.01" rpy="3.141 0.38 0"/>-->
+    <!--    </xacro:sensor_d435>-->
     <xacro:sensor_t265 name="tracking_camera" topics_ns="tracking_camera" parent="base">
         <origin xyz="0.145 0 0.1" rpy="0 -1.04 0"/>
     </xacro:sensor_t265>
+    <link name="livox_frame">
+        <collision>
+            <origin rpy="0 0 0" xyz="0 0 0"/>
+            <geometry>
+                <box size="0.01 1.0 1.0"/>
+            </geometry>
+        </collision>
+        <collision>
+            <origin rpy="0 0 0" xyz="0 0 0"/>
+            <geometry>
+                <box size="1.0 0.01 1.0"/>
+            </geometry>
+        </collision>
+    </link>
+    <joint name="livox_fixed" type="fixed">
+        <origin rpy="-2.59 1.03 3.09" xyz="0.3535 -0.057 -0.0185"/>
+        <parent link="base"/>
+        <child link="livox_frame"/>
+    </joint>
 </robot>

Commit message: Add body filter

File: legged_perceptive_description/urdf/robot.xacro (robot description, xacro)
@@ -9,5 +9,5 @@
     <!--    </xacro:sensor_d435>-->
     <xacro:sensor_t265 name="tracking_camera" topics_ns="tracking_camera" parent="base">
-        <origin xyz="0.145 0 0.1" rpy="0 -1.04 0"/>
+        <origin xyz="0.15 0 0.1" rpy="0 -1.04 0"/>
     </xacro:sensor_t265>
     <link name="livox_frame">
@@ -15,5 +15,5 @@
             <origin rpy="0 0 0" xyz="0 0 0"/>
             <geometry>
-                <box size="0.01 1.0 1.0"/>
+                <box size="0.01 5.0 5.0"/>
             </geometry>
         </collision>
@@ -21,5 +21,5 @@
             <origin rpy="0 0 0" xyz="0 0 0"/>
             <geometry>
-                <box size="1.0 0.01 1.0"/>
+                <box size="5.0 0.01 5.0"/>
             </geometry>
         </collision>

Commit message: Add another mid360

File: legged_perceptive_description/urdf/robot.xacro (robot description, xacro)
@@ -13,5 +13,5 @@
     <link name="livox_frame">
         <collision>
-            <origin rpy="0 0 0" xyz="0 0 0"/>
+            <origin rpy="-2.59 1.03 3.09" xyz="0.38 -0.057 -0.0185"/>
             <geometry>
                 <box size="0.01 5.0 5.0"/>
@@ -19,5 +19,17 @@
         </collision>
         <collision>
-            <origin rpy="0 0 0" xyz="0 0 0"/>
+            <origin rpy="-2.59 1.03 3.09" xyz="0.38 -0.057 -0.0185"/>
+            <geometry>
+                <box size="5.0 0.01 5.0"/>
+            </geometry>
+        </collision>
+        <collision>
+            <origin rpy="2.59 1.03 -3.09" xyz="0.38 0.057 -0.0185"/>
+            <geometry>
+                <box size="0.01 5.0 5.0"/>
+            </geometry>
+        </collision>
+        <collision>
+            <origin rpy="2.59 1.03 -3.09" xyz="0.38 0.057 -0.0185"/>
             <geometry>
                 <box size="5.0 0.01 5.0"/>
@@ -26,5 +38,5 @@
     </link>
     <joint name="livox_fixed" type="fixed">
-        <origin rpy="-2.59 1.03 3.09" xyz="0.3535 -0.057 -0.0185"/>
+        <origin rpy="0 0 0" xyz="0 0 0"/>
         <parent link="base"/>
         <child link="livox_frame"/>

Commit message: New link for livox

File: legged_perceptive_description/urdf/robot.xacro (robot description, xacro)
@@ -9,31 +9,7 @@
     <!--    </xacro:sensor_d435>-->
     <xacro:sensor_t265 name="tracking_camera" topics_ns="tracking_camera" parent="base">
-        <origin xyz="0.15 0 0.1" rpy="0 -1.04 0"/>
+        <origin xyz="0.16 0 0.085" rpy="0 -1.04 0"/>
     </xacro:sensor_t265>
     <link name="livox_frame">
-        <collision>
-            <origin rpy="-2.59 1.03 3.09" xyz="0.38 -0.057 -0.0185"/>
-            <geometry>
-                <box size="0.01 5.0 5.0"/>
-            </geometry>
-        </collision>
-        <collision>
-            <origin rpy="-2.59 1.03 3.09" xyz="0.38 -0.057 -0.0185"/>
-            <geometry>
-                <box size="5.0 0.01 5.0"/>
-            </geometry>
-        </collision>
-        <collision>
-            <origin rpy="2.59 1.03 -3.09" xyz="0.38 0.057 -0.0185"/>
-            <geometry>
-                <box size="0.01 5.0 5.0"/>
-            </geometry>
-        </collision>
-        <collision>
-            <origin rpy="2.59 1.03 -3.09" xyz="0.38 0.057 -0.0185"/>
-            <geometry>
-                <box size="5.0 0.01 5.0"/>
-            </geometry>
-        </collision>
     </link>
     <joint name="livox_fixed" type="fixed">
@@ -42,3 +18,37 @@
         <child link="livox_frame"/>
     </joint>
+    <link name="livox_right">
+        <collision>
+            <geometry>
+                <box size="0.003 5.0 5.0"/>
+            </geometry>
+        </collision>
+        <collision>
+            <geometry>
+                <box size="5.0 0.003 5.0"/>
+            </geometry>
+        </collision>
+    </link>
+    <joint name="livox_right_fixed" type="fixed">
+        <origin rpy="-2.59 1.03 3.09" xyz="0.365 -0.068 -0.0185"/>
+        <parent link="livox_frame"/>
+        <child link="livox_right"/>
+    </joint>
+    <link name="livox_left">
+        <collision>
+            <geometry>
+                <box size="0.003 5.0 5.0"/>
+            </geometry>
+        </collision>
+        <collision>
+            <geometry>
+                <box size="5.0 0.003 5.0"/>
+            </geometry>
+        </collision>
+    </link>
+    <joint name="livox_left_fixed" type="fixed">
+        <origin rpy="2.59 1.03 -3.09" xyz="0.365 0.068 -0.0185"/>
+        <parent link="livox_frame"/>
+        <child link="livox_left"/>
+    </joint>
 </robot>

Commit message: Add mid360.xacro

File: legged_perceptive_description/urdf/robot.xacro (robot description, xacro)
@@ -5,4 +5,5 @@
     <xacro:include filename="$(find legged_perceptive_description)/urdf/sensor_d435.xacro"/>
     <xacro:include filename="$(find legged_perceptive_description)/urdf/sensor_t265.xacro"/>
+    <xacro:include filename="$(find legged_perceptive_description)/urdf/mid360.xacro"/>
     <!--    <xacro:sensor_d435 name="front_camera" topics_ns="front_camera" parent="base">-->
     <!--        <origin xyz="0.36 -0.0 0.01" rpy="3.141 0.38 0"/>-->
@@ -11,44 +12,9 @@
         <origin xyz="0.16 0 0.085" rpy="0 -1.04 0"/>
     </xacro:sensor_t265>
-    <link name="livox_frame">
-    </link>
-    <joint name="livox_fixed" type="fixed">
-        <origin rpy="0 0 0" xyz="0 0 0"/>
-        <parent link="base"/>
-        <child link="livox_frame"/>
-    </joint>
-    <link name="livox_right">
-        <collision>
-            <geometry>
-                <box size="0.003 5.0 5.0"/>
-            </geometry>
-        </collision>
-        <collision>
-            <geometry>
-                <box size="5.0 0.003 5.0"/>
-            </geometry>
-        </collision>
-    </link>
-    <joint name="livox_right_fixed" type="fixed">
-        <origin rpy="-2.59 1.03 3.09" xyz="0.365 -0.068 -0.0185"/>
-        <parent link="livox_frame"/>
-        <child link="livox_right"/>
-    </joint>
-    <link name="livox_left">
-        <collision>
-            <geometry>
-                <box size="0.003 5.0 5.0"/>
-            </geometry>
-        </collision>
-        <collision>
-            <geometry>
-                <box size="5.0 0.003 5.0"/>
-            </geometry>
-        </collision>
-    </link>
-    <joint name="livox_left_fixed" type="fixed">
-        <origin rpy="2.59 1.03 -3.09" xyz="0.365 0.068 -0.0185"/>
-        <parent link="livox_frame"/>
-        <child link="livox_left"/>
-    </joint>
+    <xacro:mid360 name="livox_right" parent="base">
+        <origin xyz="0.365 -0.068 -0.0185" rpy="-2.59 1.03 3.09"/>
+    </xacro:mid360>
+    <xacro:mid360 name="livox_left" parent="base">
+        <origin xyz="0.365 0.068 -0.0185" rpy="2.59 1.03 -3.09"/>
+    </xacro:mid360>
 </robot>

Commit message: Update mid360 pose

File: legged_perceptive_description/urdf/robot.xacro (robot description, xacro)
@@ -13,8 +13,8 @@
     </xacro:sensor_t265>
     <xacro:mid360 name="livox_right" parent="base">
-        <origin xyz="0.365 -0.068 -0.0185" rpy="-2.59 1.03 3.09"/>
+        <origin xyz="0.365 -0.068 -0.030" rpy="-2.59 1.03 3.09"/>
     </xacro:mid360>
     <xacro:mid360 name="livox_left" parent="base">
-        <origin xyz="0.365 0.068 -0.0185" rpy="2.59 1.03 -3.09"/>
+        <origin xyz="0.365 0.068 -0.030" rpy="2.59 1.03 -3.09"/>
     </xacro:mid360>
 </robot>
